File: schematics/base_station/base_station.sch (EAGLE design)
At the start: 6 parts, among them Q1 MOSFET

Commit message: Adding schematic for logger
Changed lines of the file:
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@@
 <part name="RASPBERRY_PI_HEADER" library="SparkFun-Boards" deviceset="RASPBERRYPI-40-PIN-GPIO" device=""/>
 <part name="GND1" library="SparkFun-Aesthetics" deviceset="GND" device=""/>
-<part name="SUPPLY2" library="SparkFun-Aesthetics" deviceset="5V" device=""/>
 <part name="GND2" library="SparkFun-Aesthetics" deviceset="GND" device=""/>
 <part name="GND3" library="SparkFun-Aesthetics" deviceset="GND" device=""/>
@@
 <instance part="RASPBERRY_PI_HEADER" gate="G$1" x="157.48" y="45.72"/>
 <instance part="GND1" gate="1" x="34.29" y="22.86" rot="R180"/>
-<instance part="SUPPLY2" gate="G$1" x="25.4" y="82.55"/>
 <instance part="GND2" gate="1" x="124.46" y="11.43"/>
 <instance part="GND3" gate="1" x="110.49" y="8.89"/>
@@
 <net name="5V" class="0">
 <segment>
-<pinref part="POWER_SWITCH" gate="1" pin="O"/>
-<pinref part="SUPPLY2" gate="G$1" pin="5V"/>
-<wire x1="19.05" y1="82.55" x2="25.4" y2="82.55" width="0.1524" layer="91"/>
-</segment>
-<segment>
-<pinref part="CONTROLLER" gate="G$1" pin="PWR"/>
-<wire x1="45.72" y1="68.58" x2="38.1" y2="68.58" width="0.1524" layer="91"/>
-<label x="38.1" y="68.58" size="1.778" layer="95"/>
-</segment>
-<segment>
 <pinref part="RASPBERRY_PI_HEADER" gate="G$1" pin="5V@2"/>
 <wire x1="142.24" y1="71.12" x2="134.62" y2="71.12" width="0.1524" layer="91"/>
@@
 <pinref part="SUPPLY3" gate="G$1" pin="5V"/>
 </segment>
+<segment>
+<pinref part="POWER_SWITCH" gate="1" pin="O"/>
+<pinref part="CONTROLLER" gate="G$1" pin="PWR"/>
+<wire x1="45.72" y1="68.58" x2="36.83" y2="68.58" width="0.1524" layer="91"/>
+<wire x1="36.83" y1="68.58" x2="36.83" y2="82.55" width="0.1524" layer="91"/>
+<wire x1="36.83" y1="82.55" x2="19.05" y2="82.55" width="0.1524" layer="91"/>
+<label x="34.29" y="82.55" size="1.778" layer="95"/>
+</segment>
 </net>
